Commit message: fixed TF and visualoizations to be more accurate

File: arduinobot_ws/src/arduinobot_description/urdf/arduinobot.urdf.xacro (robot description, xacro)
@@ -25,4 +25,5 @@
     <!-- Links -->
     <link name="world" />
+    <!-- Base Link -->
     <link name="base_link">
         <visual>
@@ -30,5 +31,5 @@
                 <mesh filename="package://arduinobot_description/meshes/basement.STL" scale="0.01 0.01 0.01" />
             </geometry>
-            <origin xyz="-0.5 -0.5 0" rpy="0 0 0" /> <!-- needed in order to render the mesh properly -->
+            <origin xyz="-0.4795 -0.5 0" rpy="0 0 0" /> <!-- needed in order to render the mesh properly -->
         </visual>
         <collision>
@@ -36,8 +37,9 @@
                 <mesh filename="package://arduinobot_description/meshes/basement.STL" scale="0.01 0.01 0.01" />
             </geometry>
-            <origin xyz="-0.5 -0.5 0" rpy="0 0 0" />
-        </collision>
-        <xacro:default_inertial mass="1.0" />
-    </link>
+            <origin xyz="-0.4795 -0.5 0" rpy="0 0 0" />
+        </collision>
+        <xacro:default_inertial mass="1.0" />
+    </link>
+    <!-- Base Plate -->
     <link name="base_plate">
         <visual>
@@ -45,5 +47,5 @@
                 <mesh filename="package://arduinobot_description/meshes/base_plate.STL" scale="0.01 0.01 0.01" />
             </geometry>
-            <origin xyz="-0.39 -0.39 -0.56" rpy="0 0 0" /> <!-- needed in order to render the mesh properly -->
+            <origin xyz="-0.360 -0.405 -0.56" rpy="0 0 0" /> <!-- needed in order to render the mesh properly -->
         </visual>
         <collision>
@@ -51,8 +53,9 @@
                 <mesh filename="package://arduinobot_description/meshes/base_plate.STL" scale="0.01 0.01 0.01" />
             </geometry>
-            <origin xyz="-0.39 -0.39 -0.56" rpy="0 0 0" />
-        </collision>
-        <xacro:default_inertial mass="1.0" />
-    </link>
+            <origin xyz="-0.360 -0.405 -0.56" rpy="0 0 0" />
+        </collision>
+        <xacro:default_inertial mass="1.0" />
+    </link>
+    <!-- Forward Drive Arm -->
     <link name="forward_drive_arm_link">
         <visual>
@@ -60,5 +63,5 @@
                 <mesh filename="package://arduinobot_description/meshes/forward_drive_arm.STL" scale="0.01 0.01 0.01" />
             </geometry>
-            <origin xyz="0.19 0.06 -0.08" rpy="0 -${PI/2} ${PI/2}" /> <!-- needed in order to render the mesh properly -->
+            <origin xyz="0.18 0.075 -0.075" rpy="0 -${PI/2} ${PI/2}" /> <!-- needed in order to render the mesh properly -->
         </visual>
         <collision>
@@ -66,8 +69,9 @@
                 <mesh filename="package://arduinobot_description/meshes/forward_drive_arm.STL" scale="0.01 0.01 0.01" />
             </geometry>
-            <origin xyz="0.19 0.06 -0.08" rpy="0 -${PI/2} ${PI/2}" />
-        </collision>
-        <xacro:default_inertial mass="1.0" />
-    </link>
+            <origin xyz="0.18 0.075 -0.07" rpy="0 -${PI/2} ${PI/2}" />
+        </collision>
+        <xacro:default_inertial mass="1.0" />
+    </link>
+    <!-- Horizontal Arm -->
     <link name="horizontal_arm_link">
         <visual>
@@ -75,5 +79,5 @@
                 <mesh filename="package://arduinobot_description/meshes/horizontal_arm.STL" scale="0.01 0.01 0.01" />
             </geometry>
-            <origin xyz="-0.03 -0.4 -0.06" rpy="${PI/2} 0 ${PI/2}" /> <!-- needed in order to render the mesh properly -->
+            <origin xyz="-0.04 -0.075 -0.075" rpy="${PI/2} 0 ${PI/2}" /> <!-- needed in order to render the mesh properly -->
             </visual>
         <collision>
@@ -81,8 +85,9 @@
                 <mesh filename="package://arduinobot_description/meshes/horizontal_arm.STL" scale="0.01 0.01 0.01" />
             </geometry>
-            <origin xyz="-0.03 -0.4 -0.06" rpy="${PI/2} 0 ${PI/2}" />
-        </collision>
-        <xacro:default_inertial mass="1.0" />
-    </link>
+            <origin xyz="-0.04 -0.075 -0.075" rpy="${PI/2} 0 ${PI/2}" />
+        </collision>
+        <xacro:default_inertial mass="1.0" />
+    </link>
+    <!-- Claw Support -->
     <link name="claw_support_link">
         <visual>
@@ -90,5 +95,5 @@
                 <mesh filename="package://arduinobot_description/meshes/claw_support.STL" scale="0.01 0.01 0.01" />
             </geometry>
-            <origin xyz="0 -0.05 -0.15" rpy="0 0 ${PI/2}" /> <!-- needed in order to render the mesh properly -->
+            <origin xyz="0.128 -0.06 -0.15" rpy="0 0 ${PI/2}" /> <!-- needed in order to render the mesh properly -->
         </visual>
         <collision>
@@ -96,8 +101,9 @@
                 <mesh filename="package://arduinobot_description/meshes/claw_support.STL" scale="0.01 0.01 0.01" />
             </geometry>
-            <origin xyz="0 -0.05 -0.15" rpy="0 0 ${PI/2}" />
+            <origin xyz="0.128 -0.06 -0.15" rpy="0 0 ${PI/2}" />
         </collision>
         <xacro:default_inertial mass="0.05" />
     </link>
+    <!-- Gripper Right -->
     <link name="gripper_right_link">
         <visual>
@@ -105,5 +111,5 @@
                 <mesh filename="package://arduinobot_description/meshes/right_finger.STL" scale="0.01 0.01 0.01" />
             </geometry>
-            <origin xyz="-0.1 0.50 -0.1" rpy="0 0 -${PI/2}" /> <!-- needed in order to render the mesh properly -->
+            <origin xyz="-0.105 0.4758 -0.0925" rpy="0 0 -${PI/2}" /> <!-- needed in order to render the mesh properly -->
         </visual>
         <collision>
@@ -111,8 +117,9 @@
                 <mesh filename="package://arduinobot_description/meshes/right_finger.STL" scale="0.01 0.01 0.01" />
             </geometry>
-            <origin xyz="-0.1 0.50 -0.1" rpy="0 0 -${PI/2}" />
+            <origin xyz="-0.105 0.4758 -0.0925" rpy="0 0 -${PI/2}" />
         </collision>
         <xacro:default_inertial mass="0.01" />
     </link>
+    <!-- Gripper Left -->
     <link name="gripper_left_link">
         <visual>
@@ -120,5 +127,5 @@
                 <mesh filename="package://arduinobot_description/meshes/left_finger.STL" scale="0.01 0.01 0.01" />
             </geometry>
-            <origin xyz="-0.04 0.50 -0.1" rpy="0 0 -${PI/2}" /> <!-- needed in order to render the mesh properly -->
+            <origin xyz="-0.035 0.4758 -0.0925" rpy="0 0 -${PI/2}" /> <!-- needed in order to render the mesh properly -->
         </visual>
         <collision>
@@ -126,5 +133,5 @@
                 <mesh filename="package://arduinobot_description/meshes/left_finger.STL" scale="0.01 0.01 0.01" />
             </geometry>
-            <origin xyz="-0.04 0.50 -0.1" rpy="0 0 -${PI/2}" />
+            <origin xyz="-0.035 0.4758 -0.0925" rpy="0 0 -${PI/2}" />
         </collision>
         <xacro:default_inertial mass="0.01" />
@@ -151,44 +158,50 @@
         <origin xyz="0 0 0" rpy="0 0 0" /> <!-- needed in order to fix the base_link to the world -->
     </joint>
+    <!-- Base to Base Plate Joint (TF Transform) -->
     <joint name="joint_1" type="revolute">
-        <parent link="base_link" />
-        <child link="base_plate" />
-        <axis xyz="0 0 1" />
-        <origin xyz="0 0 0.307" rpy="0 0 0" /> <!-- needed in order to fix the base_plate to the base_link -->
-        <limit lower="-${PI/2}" upper="${PI/2}" effort="${effort}" velocity="${velocity}" />
-    </joint>
+        <parent link="base_link"/>
+        <child link="base_plate"/>
+        <origin xyz="0 0 0.31" rpy="0 0 0"/> <!-- Relative transform -->
+        <axis xyz="0 0 1"/>
+        <limit lower="-${PI/2}" upper="${PI/2}" effort="${effort}" velocity="${velocity}"/>
+    </joint>
+    <!-- Base Plate to Forward Drive Arm Joint (TF Transform) -->
     <joint name="joint_2" type="revolute">
-        <parent link="base_plate" />
-        <child link="forward_drive_arm_link" />
-        <axis xyz="1 0 0" />
-        <origin xyz="-0.02 0 0.35" rpy="0 0 0" /> <!-- needed in order to fix the forward_drive_arm to the base_plate -->
-        <limit lower="-${PI/2}" upper="${PI/2}" effort="${effort}" velocity="${velocity}" />
-    </joint>
+        <parent link="base_plate"/>
+        <child link="forward_drive_arm_link"/>
+        <origin xyz="0.018 0.0070 0.355" rpy="0 0 0"/> <!-- Relative transform -->
+        <axis xyz="1 0 0"/>
+        <limit lower="-${PI/2}" upper="${PI/2}" effort="${effort}" velocity="${velocity}"/>
+    </joint>
+    <!-- Forward Drive Arm to Horizontal Arm Joint (TF Transform) -->
     <joint name="joint_3" type="revolute">
-        <parent link="forward_drive_arm_link" />
-        <child link="horizontal_arm_link" />
-        <axis xyz="1 0 0" />
-        <origin xyz="0 0 0.8" rpy="0 0 0" /> <!-- needed in order to fix the horizontal_arm to the forward_drive_arm -->
-        <limit lower="-${PI/2}" upper="${PI/2}" effort="${effort}" velocity="${velocity}" />
-    </joint>
+        <parent link="forward_drive_arm_link"/>
+        <child link="horizontal_arm_link"/>
+        <origin xyz="0.0025 0.023 0.8" rpy="0 0 0"/> <!-- Relative transform -->
+        <axis xyz="1 0 0"/>
+        <limit lower="-${PI/2}" upper="${PI/2}" effort="${effort}" velocity="${velocity}"/>
+    </joint>
+    <!-- Horizontal Arm to Claw Support Joint (TF Transform) -->
     <joint name="horizontal_arm_to_claw_support" type="fixed">
-        <parent link="horizontal_arm_link" />
-        <child link="claw_support_link" />
-        <origin xyz="0 0.82 0" rpy="0 0 0" /> <!-- needed in order to fix the claw_support to the horizontal_arm -->
-    </joint>
+        <parent link="horizontal_arm_link"/>
+        <child link="claw_support_link"/>
+        <origin xyz="0.0 1.15 -0.001" rpy="0 0 0"/> <!-- Relative transform -->
+    </joint>
+    <!-- Claw Support to Gripper Right Joint (TF Transform) -->
     <joint name="joint_4" type="revolute">
-        <parent link="claw_support_link" />
-        <child link="gripper_right_link" />
-        <axis xyz="0 0 1" />
-        <origin xyz="-0.04 0.13 -0.1" rpy="0 0 0" /> <!-- needed in order to fix the gripper_right to the claw_support -->
-        <limit lower="-${PI/2}" upper="0.0" effort="${effort}" velocity="${velocity}" />
-    </joint>
+        <parent link="claw_support_link"/>
+        <child link="gripper_right_link"/>
+        <origin xyz="0.092 0.145 -0.09" rpy="0 0 0"/> <!-- Relative transform -->
+        <axis xyz="0 0 1"/>
+        <limit lower="-${PI/2}" upper="0" effort="${effort}" velocity="${velocity}"/>
+    </joint>
+    <!-- Claw Support to Gripper Left Joint (TF Transform) -->
     <joint name="joint_5" type="revolute">
-        <parent link="claw_support_link" />
-        <child link="gripper_left_link" />
-        <axis xyz="0 0 1" />
-        <origin xyz="-0.22 0.13 -0.1" rpy="0 0 0" /> <!-- needed in order to fix the gripper_left to the claw_support -->
-        <mimic joint="joint_4" multiplier="-1" /> <!-- needed to make the grippers move in opposite directions -->
-        <limit lower="0.0" upper="${PI/2}" effort="${effort}" velocity="${velocity}" />
+        <parent link="claw_support_link"/>
+        <child link="gripper_left_link"/>
+        <origin xyz="-0.09 0.145 -0.09" rpy="0 0 0"/> <!-- Relative transform -->
+        <axis xyz="0 0 1"/>
+        <limit lower="0" upper="${PI/2}" effort="${effort}" velocity="${velocity}"/>
+        <mimic joint="joint_4" multiplier="-1" offset="0"/>
     </joint>
     <joint name="rgb_camera_to_base_link" type="fixed">
