Commit message: fixed position for the horizontal arm

File: arduinobot_ws/install/arduinobot_description/share/arduinobot_description/urdf/arduinobot.urdf.xacro (robot description, xacro)
@@ -1,212 +1 @@
-<?xml version="1.0"?>
-<!-- ros2 launch urdf_tutorial display.launch.py model:=/home/raz/projects/manipulator-project/arduinobot_ws/src/arduinobot_description/urdf/arduinobot.urdf.xacro -->
-<robot xmlns:xacro="http://www.ros.org/wiki/xacro" name="arduinobot">
-    <!-- Start GZ or Ignition depending on ROS 2 Version -->
-    <xacro:arg name="is_ignition" default="true"/>
-    <!-- Load Simulated or Real Hardware Interfaces -->
-    <xacro:arg name="is_sim" default="true"/>
-    <!-- Include Gazebo Parameters -->
-    <xacro:include filename="$(find arduinobot_description)/urdf/arduinobot_gazebo.xacro" />
-    <!-- Include ros2 control Parameters -->
-    <xacro:include filename="$(find arduinobot_description)/urdf/arduinobot_ros2_control.xacro" />
-    <!-- Useful XACRO Variables (Properties) -->
-    <xacro:property name="PI" value="3.141592653589793" />
-    <xacro:property name="effort" value="30.0" />
-    <xacro:property name="velocity" value="10.0" />
-    <!-- Useful Macros -->
-    <xacro:macro name="default_inertial" params="mass"> <!-- not the actual inertia, just a placeholder -->
-        <inertial>
-            <mass value="${mass}" />
-            <inertia ixx="1.0" ixy="0.0" ixz="0.0"
-                     iyy="1.0" iyz="0.0"
-                     izz="1.0" />
-        </inertial>
-    </xacro:macro>
-    <!-- Links -->
-    <link name="world" />
-    <!-- Base Link -->
-    <link name="base_link">
-        <visual>
-            <geometry>
-                <mesh filename="package://arduinobot_description/meshes/basement.STL" scale="0.01 0.01 0.01" />
-            </geometry>
-            <origin xyz="-0.4795 -0.5 0" rpy="0 0 0" /> <!-- needed in order to render the mesh properly -->
-        </visual>
-        <collision>
-            <geometry>
-                <mesh filename="package://arduinobot_description/meshes/basement.STL" scale="0.01 0.01 0.01" />
-            </geometry>
-            <origin xyz="-0.4795 -0.5 0" rpy="0 0 0" />
-        </collision>
-        <xacro:default_inertial mass="1.0" />
-    </link>
-    <!-- Base Plate -->
-    <link name="base_plate">
-        <visual>
-            <geometry>
-                <mesh filename="package://arduinobot_description/meshes/base_plate.STL" scale="0.01 0.01 0.01" />
-            </geometry>
-            <origin xyz="-0.360 -0.405 -0.56" rpy="0 0 0" /> <!-- needed in order to render the mesh properly -->
-        </visual>
-        <collision>
-            <geometry>
-                <mesh filename="package://arduinobot_description/meshes/base_plate.STL" scale="0.01 0.01 0.01" />
-            </geometry>
-            <origin xyz="-0.360 -0.405 -0.56" rpy="0 0 0" />
-        </collision>
-        <xacro:default_inertial mass="1.0" />
-    </link>
-    <!-- Forward Drive Arm -->
-    <link name="forward_drive_arm_link">
-        <visual>
-            <geometry>
-                <mesh filename="package://arduinobot_description/meshes/forward_drive_arm.STL" scale="0.01 0.01 0.01" />
-            </geometry>
-            <origin xyz="0.18 0.075 -0.075" rpy="0 -${PI/2} ${PI/2}" /> <!-- needed in order to render the mesh properly -->
-        </visual>
-        <collision>
-            <geometry>
-                <mesh filename="package://arduinobot_description/meshes/forward_drive_arm.STL" scale="0.01 0.01 0.01" />
-            </geometry>
-            <origin xyz="0.18 0.075 -0.07" rpy="0 -${PI/2} ${PI/2}" />
-        </collision>
-        <xacro:default_inertial mass="1.0" />
-    </link>
-    <!-- Horizontal Arm -->
-    <link name="horizontal_arm_link">
-        <visual>
-            <geometry>
-                <mesh filename="package://arduinobot_description/meshes/horizontal_arm.STL" scale="0.01 0.01 0.01" />
-            </geometry>
-            <origin xyz="-0.04 -0.075 -0.075" rpy="${PI/2} 0 ${PI/2}" /> <!-- needed in order to render the mesh properly -->
-            </visual>
-        <collision>
-            <geometry>
-                <mesh filename="package://arduinobot_description/meshes/horizontal_arm.STL" scale="0.01 0.01 0.01" />
-            </geometry>
-            <origin xyz="-0.04 -0.075 -0.075" rpy="${PI/2} 0 ${PI/2}" />
-        </collision>
-        <xacro:default_inertial mass="1.0" />
-    </link>
-    <!-- Claw Support -->
-    <link name="claw_support_link">
-        <visual>
-            <geometry>
-                <mesh filename="package://arduinobot_description/meshes/claw_support.STL" scale="0.01 0.01 0.01" />
-            </geometry>
-            <origin xyz="0.128 -0.06 -0.15" rpy="0 0 ${PI/2}" /> <!-- needed in order to render the mesh properly -->
-        </visual>
-        <collision>
-            <geometry>
-                <mesh filename="package://arduinobot_description/meshes/claw_support.STL" scale="0.01 0.01 0.01" />
-            </geometry>
-            <origin xyz="0.128 -0.06 -0.15" rpy="0 0 ${PI/2}" />
-        </collision>
-        <xacro:default_inertial mass="0.05" />
-    </link>
-    <!-- Gripper Right -->
-    <link name="gripper_right_link">
-        <visual>
-            <geometry>
-                <mesh filename="package://arduinobot_description/meshes/right_finger.STL" scale="0.01 0.01 0.01" />
-            </geometry>
-            <origin xyz="-0.105 0.4758 -0.0925" rpy="0 0 -${PI/2}" /> <!-- needed in order to render the mesh properly -->
-        </visual>
-        <collision>
-            <geometry>
-                <mesh filename="package://arduinobot_description/meshes/right_finger.STL" scale="0.01 0.01 0.01" />
-            </geometry>
-            <origin xyz="-0.105 0.4758 -0.0925" rpy="0 0 -${PI/2}" />
-        </collision>
-        <xacro:default_inertial mass="0.01" />
-    </link>
-    <!-- Gripper Left -->
-    <link name="gripper_left_link">
-        <visual>
-            <geometry>
-                <mesh filename="package://arduinobot_description/meshes/left_finger.STL" scale="0.01 0.01 0.01" />
-            </geometry>
-            <origin xyz="-0.035 0.4758 -0.0925" rpy="0 0 -${PI/2}" /> <!-- needed in order to render the mesh properly -->
-        </visual>
-        <collision>
-            <geometry>
-                <mesh filename="package://arduinobot_description/meshes/left_finger.STL" scale="0.01 0.01 0.01" />
-            </geometry>
-            <origin xyz="-0.035 0.4758 -0.0925" rpy="0 0 -${PI/2}" />
-        </collision>
-        <xacro:default_inertial mass="0.01" />
-    </link>
-    <link name="rgb_camera">
-        <visual>
-            <geometry>
-                <mesh filename="package://arduinobot_description/meshes/pi_camera.STL" scale="0.01 0.01 0.01" />
-            </geometry>
-            <origin xyz="-0.1 0.125 0.135" rpy="-${PI/2} 0 -${PI/2}" /> <!-- needed in order to render the mesh properly -->
-        </visual>
-        <collision>
-            <geometry>
-                <mesh filename="package://arduinobot_description/meshes/pi_camera.STL" scale="0.01 0.01 0.01" />
-            </geometry>
-            <origin xyz="-0.1 0.125 0.135" rpy="-${PI/2} 0 -${PI/2}" />
-        </collision>
-        <xacro:default_inertial mass="0.001" />
-    </link>
-    <!-- Joints -->
-    <joint name="virtual_joint" type="fixed">
-        <parent link="world" />
-        <child link="base_link" />
-        <origin xyz="0 0 0" rpy="0 0 0" /> <!-- needed in order to fix the base_link to the world -->
-    </joint>
-    <!-- Base to Base Plate Joint (TF Transform) -->
-    <joint name="joint_1" type="revolute">
-        <parent link="base_link"/>
-        <child link="base_plate"/>
-        <origin xyz="0 0 0.31" rpy="0 0 0"/> <!-- Relative transform -->
-        <axis xyz="0 0 1"/>
-        <limit lower="-${PI/2}" upper="${PI/2}" effort="${effort}" velocity="${velocity}"/>
-    </joint>
-    <!-- Base Plate to Forward Drive Arm Joint (TF Transform) -->
-    <joint name="joint_2" type="revolute">
-        <parent link="base_plate"/>
-        <child link="forward_drive_arm_link"/>
-        <origin xyz="0.018 0.0070 0.355" rpy="0 0 0"/> <!-- Relative transform -->
-        <axis xyz="1 0 0"/>
-        <limit lower="-${PI/2}" upper="${PI/2}" effort="${effort}" velocity="${velocity}"/>
-    </joint>
-    <!-- Forward Drive Arm to Horizontal Arm Joint (TF Transform) -->
-    <joint name="joint_3" type="revolute">
-        <parent link="forward_drive_arm_link"/>
-        <child link="horizontal_arm_link"/>
-        <origin xyz="0.0025 0.023 0.8" rpy="0 0 0"/> <!-- Relative transform -->
-        <axis xyz="1 0 0"/>
-        <limit lower="-${PI/2}" upper="${PI/2}" effort="${effort}" velocity="${velocity}"/>
-    </joint>
-    <!-- Horizontal Arm to Claw Support Joint (TF Transform) -->
-    <joint name="horizontal_arm_to_claw_support" type="fixed">
-        <parent link="horizontal_arm_link"/>
-        <child link="claw_support_link"/>
-        <origin xyz="0.0 1.15 -0.001" rpy="0 0 0"/> <!-- Relative transform -->
-    </joint>
-    <!-- Claw Support to Gripper Right Joint (TF Transform) -->
-    <joint name="joint_4" type="revolute">
-        <parent link="claw_support_link"/>
-        <child link="gripper_right_link"/>
-        <origin xyz="0.092 0.145 -0.09" rpy="0 0 0"/> <!-- Relative transform -->
-        <axis xyz="0 0 1"/>
-        <limit lower="-${PI/2}" upper="0" effort="${effort}" velocity="${velocity}"/>
-    </joint>
-    <!-- Claw Support to Gripper Left Joint (TF Transform) -->
-    <joint name="joint_5" type="revolute">
-        <parent link="claw_support_link"/>
-        <child link="gripper_left_link"/>
-        <origin xyz="-0.09 0.145 -0.09" rpy="0 0 0"/> <!-- Relative transform -->
-        <axis xyz="0 0 1"/>
-        <limit lower="0" upper="${PI/2}" effort="${effort}" velocity="${velocity}"/>
-        <mimic joint="joint_4" multiplier="-1" offset="0"/>
-    </joint>
-    <joint name="rgb_camera_to_base_link" type="fixed">
-        <parent link="base_link" />
-        <child link="rgb_camera" />
-        <origin xyz="0 0.45 0.2" rpy="0 -0.5 ${PI/2}" /> <!-- needed in order to fix the rgb_camera to the base_link -->
-    </joint>
-</robot>
+/home/raz/projects/manipulator-project/arduinobot_ws/src/arduinobot_description/urdf/arduinobot.urdf.xacro

File: arduinobot_ws/install/arduinobot_description/share/arduinobot_description/urdf/arduinobot_gazebo.xacro (robot description, xacro)
@@ -1,46 +1 @@
-<?xml version="1.0"?>
-<robot xmlns:xacro="http://www.ros.org/wiki/xacro" name="arduinobot">
-    <!-- Gazebo Camera Plugin -->
-    <gazebo>
-        <xacro:if value="$(arg is_ignition)"> <!-- check for ros2 humble -->
-            <plugin filename="ign_ros2_control-system" name="ign_ros2_control::IgnitionROS2ControlPlugin">
-                <parameters>$(find arduinobot_controller)/config/arduinobot_controllers.yaml</parameters>
-            </plugin>
-        </xacro:if>
-        <xacro:unless value="$(arg is_ignition)"> <!-- check for ros2 humble -->
-            <plugin filename="gz_ros2_control-system" name="gz_ros2_control::GazeboSimROS2ControlPlugin">
-                <parameters>$(find arduinobot_controller)/config/arduinobot_controllers.yaml</parameters>
-            </plugin>
-        </xacro:unless>
-    </gazebo>
-    <gazebo reference="rgb_camera">
-        <sensor name="camera" type="camera">
-            <always_on>1</always_on>
-            <update_rate>30.0</update_rate>
-            <visualize>true</visualize>
-            <topic>/image_raw</topic>
-            <gz_frame_id>rgb_camera</gz_frame_id>
-            <camera name="camera">
-                <horizontal_fov>1.15</horizontal_fov>
-                <vertical_fov>0.71</vertical_fov>
-                <image>
-                    <width>2304</width>
-                    <height>1296</height>
-                    <format>R8G8B8</format>
-                </image>
-                <clip>
-                    <near>0.01</near>
-                    <far>50</far>
-                </clip>
-                <distortion>
-                    <k1>0.0</k1>
-                    <k2>0.0</k2>
-                    <k3>0.0</k3>
-                    <p1>0.0</p1>
-                    <p2>0.0</p2>
-                    <center>0.5 0.5</center>
-                </distortion>
-            </camera>
-        </sensor>
-    </gazebo>
-</robot>
+/home/raz/projects/manipulator-project/arduinobot_ws/src/arduinobot_description/urdf/arduinobot_gazebo.xacro

File: arduinobot_ws/install/arduinobot_description/share/arduinobot_description/urdf/arduinobot_ros2_control.xacro (robot description, xacro)
@@ -1,52 +1 @@
-<?xml version="1.0"?>
-<robot xmlns:xacro="http://www.ros.org/wiki/xacro" name="arduinobot">
-    <xacro:property name="PI" value="3.141592653589793" />
-    <ros2_control type="system" name="RobotSystem">
-        <xacro:if value="$(arg is_ignition)">
-            <hardware>
-                <plugin>ign_ros2_control/IgnitionSystem</plugin>
-            </hardware>
-        </xacro:if>
-        <xacro:unless value="$(arg is_ignition)"> <!-- if you are using newer version of ros else than humble -->
-            <hardware>
-                <plugin>gz_ros2_control/GazeboSimSystem</plugin>
-            </hardware>
-        </xacro:unless>
-        <joint name="joint_1">
-            <command_interface name="position">
-                <param name="min">-${PI / 2}</param>
-                <param name="max">${PI / 2}</param>
-            </command_interface>
-            <state_interface name="position"/>
-        </joint>
-        <joint name="joint_2">
-            <command_interface name="position">
-                <param name="min">-${PI / 2}</param>
-                <param name="max">${PI / 2}</param>
-            </command_interface>
-            <state_interface name="position"/>
-        </joint>
-        <joint name="joint_3">
-            <command_interface name="position">
-                <param name="min">-${PI / 2}</param>
-                <param name="max">${PI / 2}</param>
-            </command_interface>
-            <state_interface name="position"/>
-        </joint>
-        <joint name="joint_4">
-            <command_interface name="position">
-                <param name="min">-${PI / 2}</param>
-                <param name="max">0.0</param>
-            </command_interface>
-            <state_interface name="position"/>
-        </joint>
-        <joint name="joint_5"> <!-- This joint is not independent. It mimics the behaviour of the right gripper finger-->
-            <param name="mimic">joint_4</param>
-            <param name="multiplier">-1</param>
-            <command_interface name="position">
-            <param name="min">0.0</param>
-            <param name="max">${PI / 2}</param>
-            </command_interface>
-        </joint>
-    </ros2_control>
-</robot>
+/home/raz/projects/manipulator-project/arduinobot_ws/src/arduinobot_description/urdf/arduinobot_ros2_control.xacro

File: arduinobot_ws/src/arduinobot_description/urdf/arduinobot.urdf.xacro (robot description, xacro)
@@ -79,5 +79,5 @@
                 <mesh filename="package://arduinobot_description/meshes/horizontal_arm.STL" scale="0.01 0.01 0.01" />
             </geometry>
-            <origin xyz="-0.04 -0.075 -0.075" rpy="${PI/2} 0 ${PI/2}" /> <!-- needed in order to render the mesh properly -->
+            <origin xyz="-0.04 -0.425 -0.075" rpy="${PI/2} 0 ${PI/2}" /> <!-- needed in order to render the mesh properly -->
             </visual>
         <collision>
@@ -186,5 +186,5 @@
         <parent link="horizontal_arm_link"/>
         <child link="claw_support_link"/>
-        <origin xyz="0.0 1.15 -0.001" rpy="0 0 0"/> <!-- Relative transform -->
+        <origin xyz="0.0 0.8 -0.001" rpy="0 0 0"/> <!-- Relative transform -->
     </joint>
     <!-- Claw Support to Gripper Right Joint (TF Transform) -->
