Commit message: finished Section 5: Control.
changes the literal joint names to "joint_<index>" because otherwize they dont function.

File: Robotics-and-ROS-2-Learn-by-Doing-Manipulators/Section5_Control/arduinobot_ws/src/arduinobot_description/urdf/arduinobot.urdf.xacro (robot description, xacro)
@@ -19,5 +19,5 @@
         </inertial>
     </xacro:macro>
-    <xacro:macro name="default_transmission" params="number">
+    <!-- <xacro:macro name="default_transmission" params="number">
         <transmission name="transmission_${number}">
             <plugin>transmission_interface/SimpleTransmission</plugin>
@@ -27,5 +27,5 @@
             </joint>
         </transmission>
-    </xacro:macro>
+    </xacro:macro> -->
     <!-- Links -->
     <link name="world"/>
@@ -187,8 +187,8 @@
         <mimic joint="joint_4" multiplier="-1"/>
     </joint>
-    <!-- Transmissions-->
+    <!--
     <xacro:default_transmission number="1"/>
     <xacro:default_transmission number="2"/>
     <xacro:default_transmission number="3"/>
-    <xacro:default_transmission number="4"/>
+    <xacro:default_transmission number="4"/> -->
 </robot>

File: Robotics-and-ROS-2-Learn-by-Doing-Manipulators/Section5_Control/arduinobot_ws/src/arduinobot_description/urdf/arduinobot_gazebo.xacro (robot description, xacro)
@@ -3,9 +3,7 @@
     <!-- Gazebo ros2_control plugin -->
     <gazebo>
-      <plugin filename="libgazebo_ros2_control.so" name="gazebo_ros2_control">
-        <robot_param>robot_description</robot_param>
-        <robot_param_node>robot_state_publisher</robot_param_node>
-        <parameters>$(find arduinobot_controller)/config/arduinobot_controllers.yaml</parameters>
-      </plugin>
+        <plugin filename="ign_ros2_control-system" name="ign_ros2_control::IgnitionROS2ControlPlugin">
+            <parameters>$(find arduinobot_controller)/config/arduinobot_controllers.yaml</parameters>
+        </plugin>
     </gazebo>
 </robot>

File: Robotics-and-ROS-2-Learn-by-Doing-Manipulators/Section5_Control/arduinobot_ws/src/arduinobot_description/urdf/arduinobot_ros2_control.xacro (robot description, xacro)
@@ -3,7 +3,6 @@
     <ros2_control name="RobotSystem" type="system">
         <xacro:property name="PI" value="3.14159265359" />
-        <!-- ros2_control Gazebo -->
         <hardware>
-            <plugin>gazebo_ros2_control/GazeboSystem</plugin>
+            <plugin>ign_ros2_control/IgnitionSystem</plugin>
         </hardware>
         <joint name="joint_1">

File: arduinobot_ws/src/arduinobot_description/urdf/arduinobot.urdf.xacro (robot description, xacro)
@@ -8,4 +8,6 @@
     <!-- Include Gazebo Parameters -->
     <xacro:include filename="$(find arduinobot_description)/urdf/arduinobot_gazebo.xacro" />
+    <!-- Include ros2 control Parameters -->
+    <xacro:include filename="$(find arduinobot_description)/urdf/arduinobot_ros2_control.xacro" />
     <!-- Useful XACRO Variables (Properties) -->
     <xacro:property name="PI" value="3.141592653589793" />
@@ -16,6 +18,6 @@
         <inertial>
             <mass value="${mass}" />
-            <inertia ixx="1.0" ixy="0" ixz="0"
-                     iyy="1.0" iyz="0"
+            <inertia ixx="1.0" ixy="0.0" ixz="0.0"
+                     iyy="1.0" iyz="0.0"
                      izz="1.0" />
         </inertial>
@@ -149,5 +151,5 @@
         <origin xyz="0 0 0" rpy="0 0 0" /> <!-- needed in order to fix the base_link to the world -->
     </joint>
-    <joint name="base_link_to_base_plate" type="revolute">
+    <joint name="joint_1" type="revolute">
         <parent link="base_link" />
         <child link="base_plate" />
@@ -156,5 +158,5 @@
         <limit lower="-${PI/2}" upper="${PI/2}" effort="${effort}" velocity="${velocity}" />
     </joint>
-    <joint name="base_plate_to_forward_drive_arm" type="revolute">
+    <joint name="joint_2" type="revolute">
         <parent link="base_plate" />
         <child link="forward_drive_arm_link" />
@@ -163,5 +165,5 @@
         <limit lower="-${PI/2}" upper="${PI/2}" effort="${effort}" velocity="${velocity}" />
     </joint>
-    <joint name="forward_drive_arm_to_horizontal_arm" type="revolute">
+    <joint name="joint_3" type="revolute">
         <parent link="forward_drive_arm_link" />
         <child link="horizontal_arm_link" />
@@ -175,5 +177,5 @@
         <origin xyz="0 0.82 0" rpy="0 0 0" /> <!-- needed in order to fix the claw_support to the horizontal_arm -->
     </joint>
-    <joint name="claw_support_to_gripper_right" type="revolute">
+    <joint name="joint_4" type="revolute">
         <parent link="claw_support_link" />
         <child link="gripper_right_link" />
@@ -182,10 +184,10 @@
         <limit lower="-${PI/2}" upper="0.0" effort="${effort}" velocity="${velocity}" />
     </joint>
-    <joint name="claw_support_to_gripper_left" type="revolute">
+    <joint name="joint_5" type="revolute">
         <parent link="claw_support_link" />
         <child link="gripper_left_link" />
         <axis xyz="0 0 1" />
         <origin xyz="-0.22 0.13 -0.1" rpy="0 0 0" /> <!-- needed in order to fix the gripper_left to the claw_support -->
-        <mimic joint="claw_support_to_gripper_right" multiplier="-1" /> <!-- needed to make the grippers move in opposite directions -->
+        <mimic joint="joint_4" multiplier="-1" /> <!-- needed to make the grippers move in opposite directions -->
         <limit lower="0.0" upper="${PI/2}" effort="${effort}" velocity="${velocity}" />
     </joint>

File: arduinobot_ws/src/arduinobot_description/urdf/arduinobot_gazebo.xacro (robot description, xacro)
@@ -3,9 +3,14 @@
     <!-- Gazebo Camera Plugin -->
     <gazebo>
-        <xacro:if value="$(arg is_ignition)">
-            <plugin filename="ignition-gazebo-sensors-system" name="ignition::gazebo::systems::Sensors">
-                <render_engine>ogre2</render_engine>
+        <xacro:if value="$(arg is_ignition)"> <!-- check for ros2 humble -->
+            <plugin filename="ign_ros2_control-system" name="ign_ros2_control::IgnitionROS2ControlPlugin">
+                <parameters>$(find arduinobot_controller)/config/arduinobot_controllers.yaml</parameters>
             </plugin>
         </xacro:if>
+        <xacro:unless value="$(arg is_ignition)"> <!-- check for ros2 humble -->
+            <plugin filename="gz_ros2_control-system" name="gz_ros2_control::GazeboSimROS2ControlPlugin">
+                <parameters>$(find arduinobot_controller)/config/arduinobot_controllers.yaml</parameters>
+            </plugin>
+        </xacro:unless>
     </gazebo>
     <gazebo reference="rgb_camera">

Commit message: last modofication for controller configuration .yaml file

File: Robotics-and-ROS-2-Learn-by-Doing-Manipulators/Section5_Control/arduinobot_ws/src/arduinobot_description/urdf/arduinobot.urdf.xacro (robot description, xacro)
@@ -19,5 +19,5 @@
         </inertial>
     </xacro:macro>
-    <!-- <xacro:macro name="default_transmission" params="number">
+    <xacro:macro name="default_transmission" params="number">
         <transmission name="transmission_${number}">
             <plugin>transmission_interface/SimpleTransmission</plugin>
@@ -27,5 +27,5 @@
             </joint>
         </transmission>
-    </xacro:macro> -->
+    </xacro:macro>
     <!-- Links -->
     <link name="world"/>
@@ -187,8 +187,8 @@
         <mimic joint="joint_4" multiplier="-1"/>
     </joint>
-    <!--
+    <!-- Transmissions-->
     <xacro:default_transmission number="1"/>
     <xacro:default_transmission number="2"/>
     <xacro:default_transmission number="3"/>
-    <xacro:default_transmission number="4"/> -->
+    <xacro:default_transmission number="4"/>
 </robot>

Commit message: changed joints positions for gazebo simulation to respond ros control, it appeard there is a problem with small values on the x-axis for some joints

File: Robotics-and-ROS-2-Learn-by-Doing-Manipulators/Section5_Control/arduinobot_ws/src/arduinobot_description/urdf/arduinobot.urdf.xacro (robot description, xacro)
@@ -33,5 +33,5 @@
         <xacro:default_inertial mass="1.0"/>
         <visual>
-            <origin rpy="0 0 0" xyz="-0.5 -0.5 0"/>
+            <origin rpy="0 0 0" xyz="-0.4795 -0.5 0"/>
             <geometry>
                 <mesh filename="package://arduinobot_description/meshes/basement.STL" scale="0.01 0.01 0.01"/>
@@ -39,5 +39,5 @@
         </visual>
         <collision>
-            <origin rpy="0 0 0" xyz="-0.5 -0.5 0"/>
+            <origin rpy="0 0 0" xyz="-0.4795 -0.5 0"/>
             <geometry>
                 <mesh filename="package://arduinobot_description/meshes/basement.STL" scale="0.01 0.01 0.01"/>
@@ -48,5 +48,5 @@
         <xacro:default_inertial mass="0.1"/>
         <visual>
-            <origin rpy="0 0 0" xyz="-0.39 -0.39 -0.56"/>
+            <origin rpy="0 0 0" xyz="-0.360 -0.405 -0.56"/>
             <geometry>
                 <mesh filename="package://arduinobot_description/meshes/base_plate.STL" scale="0.01 0.01 0.01"/>
@@ -54,5 +54,5 @@
         </visual>
         <collision>
-            <origin rpy="0 0 0" xyz="-0.39 -0.39 -0.56"/>
+            <origin rpy="0 0 0" xyz="-0.360 -0.405 -0.56"/>
             <geometry>
                 <mesh filename="package://arduinobot_description/meshes/base_plate.STL" scale="0.01 0.01 0.01"/>
@@ -63,5 +63,5 @@
         <xacro:default_inertial mass="0.1"/>
         <visual>
-            <origin rpy=" 0 -${PI / 2} ${PI / 2}" xyz="0.19 0.06 -0.08"/>
+            <origin rpy=" 0 -${PI / 2} ${PI / 2}" xyz="0.18 0.075 -0.075"/>
             <geometry>
                 <mesh filename="package://arduinobot_description/meshes/forward_drive_arm.STL" scale="0.01 0.01 0.01"/>
@@ -69,5 +69,5 @@
         </visual>
         <collision>
-            <origin rpy=" 0 -${PI / 2} ${PI / 2}" xyz="0.19 0.06 -0.08"/>
+            <origin rpy=" 0 -${PI / 2} ${PI / 2}" xyz="0.18 0.075 -0.075"/>
             <geometry>
                 <mesh filename="package://arduinobot_description/meshes/forward_drive_arm.STL" scale="0.01 0.01 0.01"/>
@@ -78,5 +78,5 @@
         <xacro:default_inertial mass="0.1"/>
         <visual>
-            <origin rpy="${PI / 2} 0 ${PI / 2}" xyz="-0.03 -0.4 -0.06"/>
+            <origin rpy="${PI / 2} 0 ${PI / 2}" xyz="-0.04 -0.425 -0.075"/>
             <geometry>
                 <mesh filename="package://arduinobot_description/meshes/horizontal_arm.STL" scale="0.01 0.01 0.01"/>
@@ -84,5 +84,5 @@
         </visual>
         <collision>
-            <origin rpy="${PI / 2} 0 ${PI / 2}" xyz="-0.03 -0.4 -0.06"/>
+            <origin rpy="${PI / 2} 0 ${PI / 2}" xyz="-0.04 -0.425 -0.075"/>
             <geometry>
                 <mesh filename="package://arduinobot_description/meshes/horizontal_arm.STL" scale="0.01 0.01 0.01"/>
@@ -93,5 +93,5 @@
         <xacro:default_inertial mass="0.05"/>
         <visual>
-            <origin rpy="0 0 ${PI / 2}" xyz="0 -0.05 -0.15"/>
+            <origin rpy="0 0 ${PI / 2}" xyz="0.128 -0.06 -0.15"/>
             <geometry>
                 <mesh filename="package://arduinobot_description/meshes/claw_support.STL" scale="0.01 0.01 0.01"/>
@@ -99,5 +99,5 @@
         </visual>
         <collision>
-            <origin rpy="0 0 ${PI / 2}" xyz="0 -0.05 -0.15"/>
+            <origin rpy="0 0 ${PI / 2}" xyz="0.128 -0.06 -0.15"/>
             <geometry>
                 <mesh filename="package://arduinobot_description/meshes/claw_support.STL" scale="0.01 0.01 0.01"/>
@@ -108,5 +108,5 @@
         <xacro:default_inertial mass="0.01"/>
         <visual>
-            <origin rpy="0 0 -${PI / 2}" xyz="-0.1 0.50 -0.1"/>
+            <origin rpy="0 0 -${PI / 2}" xyz="-0.105 0.4758 -0.0925"/>
             <geometry>
                 <mesh filename="package://arduinobot_description/meshes/right_finger.STL" scale="0.01 0.01 0.01"/>
@@ -114,5 +114,5 @@
         </visual>
         <collision>
-            <origin rpy="0 0 -${PI / 2}" xyz="-0.1 0.50 -0.1"/>
+            <origin rpy="0 0 -${PI / 2}" xyz="-0.105 0.4758 -0.0925"/>
             <geometry>
                 <mesh filename="package://arduinobot_description/meshes/right_finger.STL" scale="0.01 0.01 0.01"/>
@@ -123,5 +123,5 @@
         <xacro:default_inertial mass="0.01"/>
         <visual>
-            <origin rpy="0 0 -${PI / 2}" xyz="-0.04 0.50 -0.1"/>
+            <origin rpy="0 0 -${PI / 2}" xyz="-0.035 0.4758 -0.0925"/>
             <geometry>
                 <mesh filename="package://arduinobot_description/meshes/left_finger.STL" scale="0.01 0.01 0.01"/>
@@ -129,5 +129,5 @@
         </visual>
         <collision>
-            <origin rpy="0 0 -${PI / 2}" xyz="-0.04 0.50 -0.1"/>
+            <origin rpy="0 0 -${PI / 2}" xyz="-0.035 0.4758 -0.0925"/>
             <geometry>
                 <mesh filename="package://arduinobot_description/meshes/left_finger.STL" scale="0.01 0.01 0.01"/>
@@ -144,5 +144,5 @@
         <parent link="base_link"/>
         <child link = "base_plate"/>
-        <origin xyz="0 0 0.307"/>
+        <origin xyz="0 0 0.31"/>
         <axis xyz="0 0 1"/>
         <limit lower="-${PI / 2}" upper="${PI / 2}"
@@ -152,5 +152,5 @@
         <parent link="base_plate"/>
         <child link = "forward_drive_arm"/>
-        <origin xyz="-0.02 0 0.35"/>
+        <origin xyz="0.012 0.0070 0.355"/>
         <axis xyz="1 0 0"/>
         <limit lower="-${PI / 2}" upper="${PI / 2}"
@@ -168,10 +168,10 @@
         <parent link="horizontal_arm"/>
         <child link = "claw_support"/>
-        <origin xyz="0 0.82 0"/>
+        <origin xyz="0 0.8 0"/>
     </joint>
     <joint name ="joint_4" type="revolute">
         <parent link="claw_support"/>
         <child link = "gripper_right"/>
-        <origin xyz="-0.04 0.13 -0.1"/>
+        <origin xyz="0.09 0.145 -0.09"/>
         <axis xyz="0 0 1"/>
         <limit lower="-${PI / 2}" upper="0.0"
@@ -181,5 +181,5 @@
         <parent link="claw_support"/>
         <child link = "gripper_left"/>
-        <origin xyz="-0.22 0.13 -0.1"/>
+        <origin xyz="-0.09 0.145 -0.09"/>
         <axis xyz="0 0 1"/>
         <limit lower="0.0" upper="${PI / 2}"

File: Robotics-and-ROS-2-Learn-by-Doing-Manipulators/Section5_Control/arduinobot_ws/src/arduinobot_description/urdf/arduinobot_ros2_control.xacro (robot description, xacro)
@@ -2,5 +2,5 @@
 <robot xmlns:xacro="http://www.ros.org/wiki/xacro" name="arduinobot">
     <ros2_control name="RobotSystem" type="system">
-        <xacro:property name="PI" value="3.14159265359" />
+        <xacro:property name="PI" value="3.141592653589793" />
         <hardware>
             <plugin>ign_ros2_control/IgnitionSystem</plugin>

File: arduinobot_ws/src/arduinobot_description/urdf/arduinobot.urdf.xacro (robot description, xacro)
@@ -1,4 +1,3 @@
 <?xml version="1.0"?>
-<!-- ros2 launch urdf_tutorial display.launch.py model:=/home/raz/projects/manipulator-project/arduinobot_ws/src/arduinobot_description/urdf/arduinobot.urdf.xacro -->
 <robot xmlns:xacro="http://www.ros.org/wiki/xacro" name="arduinobot">
     <!-- Start GZ or Ignition depending on ROS 2 Version -->
@@ -69,5 +68,5 @@
                 <mesh filename="package://arduinobot_description/meshes/forward_drive_arm.STL" scale="0.01 0.01 0.01" />
             </geometry>
-            <origin xyz="0.18 0.075 -0.07" rpy="0 -${PI/2} ${PI/2}" />
+            <origin xyz="0.18 0.075 -0.075" rpy="0 -${PI/2} ${PI/2}" />
         </collision>
         <xacro:default_inertial mass="1.0" />
@@ -85,5 +84,5 @@
                 <mesh filename="package://arduinobot_description/meshes/horizontal_arm.STL" scale="0.01 0.01 0.01" />
             </geometry>
-            <origin xyz="-0.04 -0.075 -0.075" rpy="${PI/2} 0 ${PI/2}" />
+            <origin xyz="-0.04 -0.425 -0.075" rpy="${PI/2} 0 ${PI/2}" />
         </collision>
         <xacro:default_inertial mass="1.0" />
@@ -170,5 +169,5 @@
         <parent link="base_plate"/>
         <child link="forward_drive_arm_link"/>
-        <origin xyz="0.018 0.0070 0.355" rpy="0 0 0"/> <!-- Relative transform -->
+        <origin xyz="0 0.007 0.355" rpy="0 0 0"/> <!-- Relative transform -->
         <axis xyz="1 0 0"/>
         <limit lower="-${PI/2}" upper="${PI/2}" effort="${effort}" velocity="${velocity}"/>
@@ -178,5 +177,5 @@
         <parent link="forward_drive_arm_link"/>
         <child link="horizontal_arm_link"/>
-        <origin xyz="0.0025 0.023 0.8" rpy="0 0 0"/> <!-- Relative transform -->
+        <origin xyz="0 0.023 0.8" rpy="0 0 0"/> <!-- Relative transform -->
         <axis xyz="1 0 0"/>
         <limit lower="-${PI/2}" upper="${PI/2}" effort="${effort}" velocity="${velocity}"/>
@@ -186,5 +185,5 @@
         <parent link="horizontal_arm_link"/>
         <child link="claw_support_link"/>
-        <origin xyz="0.0 0.8 -0.001" rpy="0 0 0"/> <!-- Relative transform -->
+        <origin xyz="0.0 0.8 0" rpy="0 0 0"/> <!-- Relative transform -->
     </joint>
     <!-- Claw Support to Gripper Right Joint (TF Transform) -->
@@ -192,5 +191,5 @@
         <parent link="claw_support_link"/>
         <child link="gripper_right_link"/>
-        <origin xyz="0.092 0.145 -0.09" rpy="0 0 0"/> <!-- Relative transform -->
+        <origin xyz="0.09 0.145 -0.09" rpy="0 0 0"/> <!-- Relative transform -->
         <axis xyz="0 0 1"/>
         <limit lower="-${PI/2}" upper="0.0" effort="${effort}" velocity="${velocity}"/>

File: arduinobot_ws/src/arduinobot_description/urdf/arduinobot_gazebo.xacro (robot description, xacro)
@@ -26,5 +26,5 @@
             <update_rate>30.0</update_rate>
             <visualize>true</visualize>
-            <topic>/image_raw</topic>
+            <topic>/rgb_camera/image_raw</topic>
             <gz_frame_id>/rgb_camera</gz_frame_id>
             <camera name="camera">

File: arduinobot_ws/src/arduinobot_description/urdf/arduinobot_ros2_control.xacro (robot description, xacro)
@@ -1,20 +1,13 @@
 <?xml version="1.0"?>
 <robot xmlns:xacro="http://www.ros.org/wiki/xacro" name="arduinobot">
-    <xacro:property name="PI" value="3.141592653589793" />
-    <ros2_control type="system" name="RobotSystem">
-        <xacro:if value="$(arg is_ignition)">
-            <hardware>
-                <plugin>ign_ros2_control/IgnitionSystem</plugin>
-            </hardware>
-        </xacro:if>
-        <xacro:unless value="$(arg is_ignition)"> <!-- if you are using newer version of ros else than humble -->
-            <hardware>
-                <plugin>gz_ros2_control/GazeboSimSystem</plugin>
-            </hardware>
-        </xacro:unless>
+    <ros2_control name="RobotSystem" type="system">
+        <xacro:property name="PI" value="3.141592653589793" />
+        <hardware>
+            <plugin>ign_ros2_control/IgnitionSystem</plugin>
+        </hardware>
         <joint name="joint_1">
             <command_interface name="position">
-                <param name="min">-${PI / 2}</param>
-                <param name="max">${PI / 2}</param>
+            <param name="min">-${PI / 2}</param>
+            <param name="max">${PI / 2}</param>
             </command_interface>
             <state_interface name="position"/>
@@ -22,6 +15,6 @@
         <joint name="joint_2">
             <command_interface name="position">
-                <param name="min">-${PI / 2}</param>
-                <param name="max">${PI / 2}</param>
+            <param name="min">-${PI / 2}</param>
+            <param name="max">${PI / 2}</param>
             </command_interface>
             <state_interface name="position"/>
@@ -29,6 +22,6 @@
         <joint name="joint_3">
             <command_interface name="position">
-                <param name="min">-${PI / 2}</param>
-                <param name="max">${PI / 2}</param>
+            <param name="min">-${PI / 2}</param>
+            <param name="max">${PI / 2}</param>
             </command_interface>
             <state_interface name="position"/>
@@ -36,10 +29,10 @@
         <joint name="joint_4">
             <command_interface name="position">
-                <param name="min">-${PI / 2}</param>
-                <param name="max">0.0</param>
+            <param name="min">-${PI / 2}</param>
+            <param name="max">0.0</param>
             </command_interface>
             <state_interface name="position"/>
         </joint>
-        <joint name="joint_5"> <!-- This joint is not independent. It mimics the behaviour of the right gripper finger-->
+        <joint name="joint_5">
             <param name="mimic">joint_4</param>
             <param name="multiplier">-1</param>
