Commit message: Section 4: Digital Twin - Completed

File: arduinobot_ws/src/arduinobot_description/urdf/arduinobot.urdf.xacro (robot description, xacro)
@@ -1,7 +1,16 @@
 <?xml version="1.0"?>
+<!-- ros2 launch urdf_tutorial display.launch.py model:=/home/raz/projects/manipulator-project/arduinobot_ws/src/arduinobot_description/urdf/arduinobot.urdf.xacro -->
 <robot xmlns:xacro="http://www.ros.org/wiki/xacro" name="arduinobot">
     <xacro:property name="PI" value="3.141592653589793" />
     <xacro:property name="effort" value="30.0" />
     <xacro:property name="velocity" value="10.0" />
+    <xacro:macro name="default_inertial" params="mass"> <!-- not the actual inertia, just a placeholder -->
+        <inertial>
+            <mass value="${mass}" />
+            <inertia ixx="1.0" ixy="0" ixz="0"
+                     iyy="1.0" iyz="0"
+                     izz="1.0" />
+        </inertial>
+    </xacro:macro>
     <link name="world" />
     <link name="base_link">
@@ -12,4 +21,11 @@
             <origin xyz="-0.5 -0.5 0" rpy="0 0 0" /> <!-- needed in order to render the mesh properly -->
         </visual>
+        <collision>
+            <geometry>
+                <mesh filename="package://arduinobot_description/meshes/basement.STL" scale="0.01 0.01 0.01" />
+            </geometry>
+            <origin xyz="-0.5 -0.5 0" rpy="0 0 0" />
+        </collision>
+        <xacro:default_inertial mass="1.0" />
     </link>
     <link name="base_plate">
@@ -20,4 +36,11 @@
             <origin xyz="-0.39 -0.39 -0.56" rpy="0 0 0" /> <!-- needed in order to render the mesh properly -->
         </visual>
+        <collision>
+            <geometry>
+                <mesh filename="package://arduinobot_description/meshes/base_plate.STL" scale="0.01 0.01 0.01" />
+            </geometry>
+            <origin xyz="-0.39 -0.39 -0.56" rpy="0 0 0" />
+        </collision>
+        <xacro:default_inertial mass="1.0" />
     </link>
     <link name="forward_drive_arm_link">
@@ -28,4 +51,11 @@
             <origin xyz="0.19 0.06 -0.08" rpy="0 -${PI/2} ${PI/2}" /> <!-- needed in order to render the mesh properly -->
         </visual>
+        <collision>
+            <geometry>
+                <mesh filename="package://arduinobot_description/meshes/forward_drive_arm.STL" scale="0.01 0.01 0.01" />
+            </geometry>
+            <origin xyz="0.19 0.06 -0.08" rpy="0 -${PI/2} ${PI/2}" />
+        </collision>
+        <xacro:default_inertial mass="1.0" />
     </link>
     <link name="horizontal_arm_link">
@@ -35,5 +65,12 @@
             </geometry>
             <origin xyz="-0.03 -0.4 -0.06" rpy="${PI/2} 0 ${PI/2}" /> <!-- needed in order to render the mesh properly -->
-        </visual>
+            </visual>
+        <collision>
+            <geometry>
+                <mesh filename="package://arduinobot_description/meshes/horizontal_arm.STL" scale="0.01 0.01 0.01" />
+            </geometry>
+            <origin xyz="-0.03 -0.4 -0.06" rpy="${PI/2} 0 ${PI/2}" />
+        </collision>
+        <xacro:default_inertial mass="1.0" />
     </link>
     <link name="claw_support_link">
@@ -44,4 +81,11 @@
             <origin xyz="0 -0.05 -0.15" rpy="0 0 ${PI/2}" /> <!-- needed in order to render the mesh properly -->
         </visual>
+        <collision>
+            <geometry>
+                <mesh filename="package://arduinobot_description/meshes/claw_support.STL" scale="0.01 0.01 0.01" />
+            </geometry>
+            <origin xyz="0 -0.05 -0.15" rpy="0 0 ${PI/2}" />
+        </collision>
+        <xacro:default_inertial mass="0.05" />
     </link>
     <link name="gripper_right_link">
@@ -52,4 +96,11 @@
             <origin xyz="-0.1 0.50 -0.1" rpy="0 0 -${PI/2}" /> <!-- needed in order to render the mesh properly -->
         </visual>
+        <collision>
+            <geometry>
+                <mesh filename="package://arduinobot_description/meshes/right_finger.STL" scale="0.01 0.01 0.01" />
+            </geometry>
+            <origin xyz="-0.1 0.50 -0.1" rpy="0 0 -${PI/2}" />
+        </collision>
+        <xacro:default_inertial mass="0.01" />
     </link>
     <link name="gripper_left_link">
@@ -60,4 +111,26 @@
             <origin xyz="-0.04 0.50 -0.1" rpy="0 0 -${PI/2}" /> <!-- needed in order to render the mesh properly -->
         </visual>
+        <collision>
+            <geometry>
+                <mesh filename="package://arduinobot_description/meshes/left_finger.STL" scale="0.01 0.01 0.01" />
+            </geometry>
+            <origin xyz="-0.04 0.50 -0.1" rpy="0 0 -${PI/2}" />
+        </collision>
+        <xacro:default_inertial mass="0.01" />
+    </link>
+    <link name="rgb_camera">
+        <visual>
+            <geometry>
+                <mesh filename="package://arduinobot_description/meshes/pi_camera.STL" scale="0.01 0.01 0.01" />
+            </geometry>
+            <origin xyz="-0.1 0.125 0.135" rpy="-${PI/2} 0 -${PI/2}" /> <!-- needed in order to render the mesh properly -->
+        </visual>
+        <collision>
+            <geometry>
+                <mesh filename="package://arduinobot_description/meshes/pi_camera.STL" scale="0.01 0.01 0.01" />
+            </geometry>
+            <origin xyz="-0.1 0.125 0.135" rpy="-${PI/2} 0 -${PI/2}" />
+        </collision>
+        <xacro:default_inertial mass="0.001" />
     </link>
     <!-- Joints -->
@@ -108,3 +181,37 @@
         <limit lower="0.0" upper="${PI/2}" effort="${effort}" velocity="${velocity}" />
     </joint>
+    <joint name="rgb_camera_to_base_link" type="fixed">
+        <parent link="base_link" />
+        <child link="rgb_camera" />
+        <origin xyz="0 0.45 0.2" rpy="0 -0.5 ${PI/2}" /> <!-- needed in order to fix the rgb_camera to the base_link -->
+    </joint>
+    <!-- Gazebo Camera Plugin -->
+    <gazebo reference="rgb_camera">
+        <sensor type="camera" name="rgb_camera">
+            <always_on>true</always_on>
+            <update_rate>30.0</update_rate>
+          <camera name="rgb_camera">
+            <horizontal_fov>1.15</horizontal_fov>
+            <vertical_fov>0.71</vertical_fov>
+            <image>
+                <width>2304</width>
+                <height>1296</height>
+                <format>R8G8B8</format>
+            </image>
+            <clip>
+                <near>0.01</near>
+                <far>50</far>
+            </clip>
+          </camera>
+          <plugin name="camera_controller" filename="libgazebo_ros_camera.so">
+            <ros>
+              <remapping>image_raw:=image_raw</remapping>
+              <remapping>camera_info:=camera_info</remapping>
+            </ros>
+            <camera_name>rgb_camera</camera_name>
+            <frame_name>rgb_camera</frame_name>
+            <hack_baseline>0.07</hack_baseline>
+            </plugin>
+        </sensor>
+    </gazebo>
 </robot>

Commit message: minor

File: arduinobot_ws/src/arduinobot_description/urdf/arduinobot.urdf.xacro (robot description, xacro)
@@ -194,5 +194,5 @@
         <origin xyz="0.092 0.145 -0.09" rpy="0 0 0"/> <!-- Relative transform -->
         <axis xyz="0 0 1"/>
-        <limit lower="-${PI/2}" upper="0" effort="${effort}" velocity="${velocity}"/>
+        <limit lower="-${PI/2}" upper="0.0" effort="${effort}" velocity="${velocity}"/>
     </joint>
     <!-- Claw Support to Gripper Left Joint (TF Transform) -->
@@ -202,5 +202,5 @@
         <origin xyz="-0.09 0.145 -0.09" rpy="0 0 0"/> <!-- Relative transform -->
         <axis xyz="0 0 1"/>
-        <limit lower="0" upper="${PI/2}" effort="${effort}" velocity="${velocity}"/>
+        <limit lower="0.0" upper="${PI/2}" effort="${effort}" velocity="${velocity}"/>
         <mimic joint="joint_4" multiplier="-1" offset="0"/>
     </joint>

File: arduinobot_ws/src/arduinobot_description/urdf/arduinobot_gazebo.xacro (robot description, xacro)
@@ -1,5 +1,5 @@
 <?xml version="1.0"?>
 <robot xmlns:xacro="http://www.ros.org/wiki/xacro" name="arduinobot">
-    <!-- Gazebo Camera Plugin -->
+    <!-- Gazebo Control Plugin -->
     <gazebo>
         <xacro:if value="$(arg is_ignition)"> <!-- check for ros2 humble -->
@@ -14,14 +14,20 @@
         </xacro:unless>
     </gazebo>
+    <!-- Gazebo Camera Plugin -->
+    <gazebo>
+        <!-- ROS 2 Humble -->
+        <plugin filename="ignition-gazebo-sensors-system" name="ignition::gazebo::systems::Sensors">
+            <render_engine>ogre2</render_engine>
+        </plugin>
+    </gazebo>
     <gazebo reference="rgb_camera">
         <sensor name="camera" type="camera">
-            <always_on>1</always_on>
+            <always_on>true</always_on>
             <update_rate>30.0</update_rate>
             <visualize>true</visualize>
             <topic>/image_raw</topic>
-            <gz_frame_id>rgb_camera</gz_frame_id>
+            <gz_frame_id>/rgb_camera</gz_frame_id>
             <camera name="camera">
-                <horizontal_fov>1.15</horizontal_fov>
-                <vertical_fov>0.71</vertical_fov>
+                <horizontal_fov>1.21126</horizontal_fov>
                 <image>
                     <width>2304</width>
@@ -29,8 +35,4 @@
                     <format>R8G8B8</format>
                 </image>
-                <clip>
-                    <near>0.01</near>
-                    <far>50</far>
-                </clip>
                 <distortion>
                     <k1>0.0</k1>

Commit message: Done Section 6: Kinematics

File: arduinobot_ws/src/arduinobot_description/urdf/arduinobot.urdf.xacro (robot description, xacro)
@@ -62,5 +62,5 @@
                 <mesh filename="package://arduinobot_description/meshes/forward_drive_arm.STL" scale="0.01 0.01 0.01" />
             </geometry>
-            <origin xyz="0.18 0.075 -0.075" rpy="0 -${PI/2} ${PI/2}" /> <!-- needed in order to render the mesh properly -->
+            <origin xyz="0.2 0.075 -0.075" rpy="0 -${PI/2} ${PI/2}" /> <!-- needed in order to render the mesh properly -->
         </visual>
         <collision>
@@ -68,5 +68,5 @@
                 <mesh filename="package://arduinobot_description/meshes/forward_drive_arm.STL" scale="0.01 0.01 0.01" />
             </geometry>
-            <origin xyz="0.18 0.075 -0.075" rpy="0 -${PI/2} ${PI/2}" />
+            <origin xyz="0.2 0.075 -0.075" rpy="0 -${PI/2} ${PI/2}" />
         </collision>
         <xacro:default_inertial mass="1.0" />
@@ -177,5 +177,5 @@
         <parent link="forward_drive_arm_link"/>
         <child link="horizontal_arm_link"/>
-        <origin xyz="0 0.023 0.8" rpy="0 0 0"/> <!-- Relative transform -->
+        <origin xyz="0.0225 0.023 0.8" rpy="0 0 0"/> <!-- Relative transform -->
         <axis xyz="1 0 0"/>
         <limit lower="-${PI/2}" upper="${PI/2}" effort="${effort}" velocity="${velocity}"/>
@@ -191,5 +191,5 @@
         <parent link="claw_support_link"/>
         <child link="gripper_right_link"/>
-        <origin xyz="0.09 0.145 -0.09" rpy="0 0 0"/> <!-- Relative transform -->
+        <origin xyz="0.0915 0.145 -0.09" rpy="0 0 0"/> <!-- Relative transform -->
         <axis xyz="0 0 1"/>
         <limit lower="-${PI/2}" upper="0.0" effort="${effort}" velocity="${velocity}"/>
@@ -199,5 +199,5 @@
         <parent link="claw_support_link"/>
         <child link="gripper_left_link"/>
-        <origin xyz="-0.09 0.145 -0.09" rpy="0 0 0"/> <!-- Relative transform -->
+        <origin xyz="-0.0915 0.145 -0.09" rpy="0 0 0"/> <!-- Relative transform -->
         <axis xyz="0 0 1"/>
         <limit lower="0.0" upper="${PI/2}" effort="${effort}" velocity="${velocity}"/>

File: arduinobot_ws/src/arduinobot_description/urdf/arduinobot_gazebo.xacro (robot description, xacro)
@@ -16,5 +16,4 @@
     <!-- Gazebo Camera Plugin -->
     <gazebo>
-        <!-- ROS 2 Humble -->
         <plugin filename="ignition-gazebo-sensors-system" name="ignition::gazebo::systems::Sensors">
             <render_engine>ogre2</render_engine>

Commit message: Done Section 8: Alexa Integration

File: arduinobot_ws/src/arduinobot_description/urdf/arduinobot.urdf.xacro (robot description, xacro)
@@ -30,5 +30,8 @@
                 <mesh filename="package://arduinobot_description/meshes/basement.STL" scale="0.01 0.01 0.01" />
             </geometry>
-            <origin xyz="-0.4795 -0.5 0" rpy="0 0 0" /> <!-- needed in order to render the mesh properly -->
+            <origin xyz="-0.4795 -0.5 0" rpy="0 0 0" />
+            <material name="black">
+                <color rgba="0.05 0.05 0.05 1"/>
+            </material>
         </visual>
         <collision>
@@ -46,5 +49,8 @@
                 <mesh filename="package://arduinobot_description/meshes/base_plate.STL" scale="0.01 0.01 0.01" />
             </geometry>
-            <origin xyz="-0.360 -0.405 -0.56" rpy="0 0 0" /> <!-- needed in order to render the mesh properly -->
+            <origin xyz="-0.360 -0.405 -0.56" rpy="0 0 0" />
+            <material name="black">
+                <color rgba="0.05 0.05 0.05 1"/>
+            </material>
         </visual>
         <collision>
@@ -62,5 +68,8 @@
                 <mesh filename="package://arduinobot_description/meshes/forward_drive_arm.STL" scale="0.01 0.01 0.01" />
             </geometry>
-            <origin xyz="0.2 0.075 -0.075" rpy="0 -${PI/2} ${PI/2}" /> <!-- needed in order to render the mesh properly -->
+            <origin xyz="0.2 0.075 -0.075" rpy="0 -${PI/2} ${PI/2}" />
+            <material name="black">
+                <color rgba="0.05 0.05 0.05 1"/>
+            </material>
         </visual>
         <collision>
@@ -78,6 +87,9 @@
                 <mesh filename="package://arduinobot_description/meshes/horizontal_arm.STL" scale="0.01 0.01 0.01" />
             </geometry>
-            <origin xyz="-0.04 -0.425 -0.075" rpy="${PI/2} 0 ${PI/2}" /> <!-- needed in order to render the mesh properly -->
-            </visual>
+            <origin xyz="-0.04 -0.425 -0.075" rpy="${PI/2} 0 ${PI/2}" />
+            <material name="black">
+                <color rgba="0.05 0.05 0.05 1"/>
+            </material>
+        </visual>
         <collision>
             <geometry>
@@ -94,5 +106,8 @@
                 <mesh filename="package://arduinobot_description/meshes/claw_support.STL" scale="0.01 0.01 0.01" />
             </geometry>
-            <origin xyz="0.128 -0.06 -0.15" rpy="0 0 ${PI/2}" /> <!-- needed in order to render the mesh properly -->
+            <origin xyz="0.128 -0.06 -0.15" rpy="0 0 ${PI/2}" />
+            <material name="black">
+                <color rgba="0.05 0.05 0.05 1"/>
+            </material>
         </visual>
         <collision>
@@ -110,5 +125,8 @@
                 <mesh filename="package://arduinobot_description/meshes/right_finger.STL" scale="0.01 0.01 0.01" />
             </geometry>
-            <origin xyz="-0.105 0.4758 -0.0925" rpy="0 0 -${PI/2}" /> <!-- needed in order to render the mesh properly -->
+            <origin xyz="-0.105 0.4758 -0.0925" rpy="0 0 -${PI/2}" />
+            <material name="black">
+                <color rgba="0.05 0.05 0.05 1"/>
+            </material>
         </visual>
         <collision>
@@ -126,5 +144,8 @@
                 <mesh filename="package://arduinobot_description/meshes/left_finger.STL" scale="0.01 0.01 0.01" />
             </geometry>
-            <origin xyz="-0.035 0.4758 -0.0925" rpy="0 0 -${PI/2}" /> <!-- needed in order to render the mesh properly -->
+            <origin xyz="-0.035 0.4758 -0.0925" rpy="0 0 -${PI/2}" />
+            <material name="black">
+                <color rgba="0.05 0.05 0.05 1"/>
+            </material>
         </visual>
         <collision>
@@ -142,4 +163,7 @@
             </geometry>
             <origin xyz="-0.1 0.125 0.135" rpy="-${PI/2} 0 -${PI/2}" /> <!-- needed in order to render the mesh properly -->
+            <material name="black">
+                <color rgba="0.05 0.05 0.05 1"/>
+            </material>
         </visual>
         <collision>
