Commit message: Done Section 9: Build The Robot

File: arduinobot_ws/src/arduinobot_description/urdf/arduinobot_ros2_control.xacro (robot description, xacro)
@@ -3,7 +3,25 @@
     <ros2_control name="RobotSystem" type="system">
         <xacro:property name="PI" value="3.141592653589793" />
-        <hardware>
-            <plugin>ign_ros2_control/IgnitionSystem</plugin>
-        </hardware>
+        <!-- ros2 control Gazebo -->
+        <xacro:if value="$(arg is_sim)">
+            <hardware>
+                <plugin>ign_ros2_control/IgnitionSystem</plugin>
+            </hardware>
+            <joint name="joint_5">
+                <param name="mimic">joint_4</param>
+                <param name="multiplier">-1</param>
+                <command_interface name="position">
+                <param name="min">0.0</param>
+                <param name="max">${PI / 2}</param>
+                </command_interface>
+            </joint>
+            <!-- Joint 5 is needed only for the simulation -->
+        </xacro:if>
+        <xacro:unless value="$(arg is_sim)">
+            <hardware>
+                <plugin>arduinobot_controller?ArduinoInterface</plugin>
+                <param name="port">/dev/ttyUSB0</param>
+            </hardware>
+        </xacro:unless>
         <joint name="joint_1">
             <command_interface name="position">
@@ -34,12 +52,4 @@
             <state_interface name="position"/>
         </joint>
-        <joint name="joint_5">
-            <param name="mimic">joint_4</param>
-            <param name="multiplier">-1</param>
-            <command_interface name="position">
-            <param name="min">0.0</param>
-            <param name="max">${PI / 2}</param>
-            </command_interface>
-        </joint>
     </ros2_control>
 </robot>
